Commit message: replace stl models

File: dobot/urdf/robot1.urdf (robot description, URDF)
Before this commit: robot dobot, 8 links, 7 joints
Links:
- link link_1: geometry visual mesh filename=package://dobot/urdf/meshes/1part.stl scale=0.001 0.001 0.001
- link link_2: geometry visual mesh filename=package://dobot/urdf/meshes/2.stl scale=0.001 0.001 0.001
- link link_3: geometry visual mesh filename=package://dobot/urdf/meshes/3.stl scale=0.001 0.001 0.001
- link link_4: geometry visual mesh filename=package://dobot/urdf/meshes/raborg.stl scale=0.001 0.001 0.001

File: dobot/urdf/robot1.urdf.xacro (robot description, xacro)
@@ -22,5 +22,5 @@
         <mesh filename="package://dobot/urdf/meshes/1part.stl" scale="0.01 0.01 0.01"/>
       </geometry>
-      <material name="black"/>
+      <material name="white"/>
     </visual>
   </link>
